File: _autosave-rc-plane.kicad_sch (KiCad schematic)
At the start: 104 parts, among them J1 POWER, J2 ARMING_PLUG, J3 SMA, J4 E-MATCH_DROGUE, J5 SWD, J6 E-MATCH_RECOVERY, J8 E-MATCH_BACKUP, J9 HTSW-109-08-T-T-RA, Q1 Q_NMOS_GSD, Q2 Q_NMOS_GSD, Q3 BC547, Q4 Q_NMOS_GSD, Q5 Q_NMOS_GSD, Q6 Q_NMOS_GSD, Q7 Q_NMOS_GSD, U10 RASPBERRY_PI_4B_4GB, U8 BMM350, U9 USBLC6-2SC6, Y1 16MHz

Commit message: layout mostly done
Parts:
- removed R22: 10k, Resistor_SMD:R_0603_1608Metric, symbol Device:R_Small_US
Other:
- note removed: "Reset Pin cannot be driven HIGH"
Changed lines of the file:
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@@
 		)
 	)
-	(text "Reset Pin\ncannot be\ndriven HIGH"
-		(exclude_from_sim no)
-		(at 306.832 30.734 0)
-		(effects
-			(font
-				(size 1.27 1.27)
-			)
-			(justify left bottom)
-		)
-	)
 	(text "SPI2\n"
 		(exclude_from_sim no)
@@
 	(wire
 		(pts
-			(xy 304.8 31.75) (xy 304.8 33.02)
-		)
-		(stroke
-			(width 0)
-			(type default)
-		)
-	)
-	(wire
-		(pts
 			(xy 290.83 204.47) (xy 287.02 204.47)
 		)
@@
 	(wire
 		(pts
-			(xy 304.8 33.02) (xy 306.07 33.02)
-		)
-		(stroke
-			(width 0)
-			(type default)
-		)
-	)
-	(wire
-		(pts
 			(xy 154.94 246.38) (xy 177.8 246.38)
 		)
@@
 		)
 	)
-	(global_label "GPS_RESET"
-		(shape input)
-		(at 306.07 33.02 0)
-		(fields_autoplaced yes)
-		(effects
-			(font
-				(size 1.27 1.27)
-			)
-			(justify left)
-		)
-		(property "Intersheetrefs" "${INTERSHEET_REFS}"
-			(at 319.5174 33.02 0)
-			(effects
-				(font
-					(size 1.27 1.27)
-				)
-				(justify left)
-				(hide yes)
-			)
-		)
-	)
 	(global_label "VBUS"
 		(shape input)
@@
 	)
 	(symbol
-		(lib_id "Device:R_Small_US")
-		(at 304.8 29.21 0)
-		(unit 1)
-		(exclude_from_sim no)
-		(in_bom yes)
-		(on_board yes)
-		(dnp no)
-		(property "Reference" "R22"
-			(at 299.72 31.75 0)
-			(effects
-				(font
-					(size 1.27 1.27)
-				)
-				(justify left)
-			)
-		)
-		(property "Value" "10k"
-			(at 299.72 29.21 0)
-			(effects
-				(font
-					(size 1.27 1.27)
-				)
-				(justify left)
-			)
-		)
-		(property "Footprint" "Resistor_SMD:R_0603_1608Metric"
-			(at 304.8 29.21 0)
-			(effects
-				(font
-					(size 1.27 1.27)
-				)
-				(hide yes)
-			)
-		)
-		(property "Datasheet" "~"
-			(at 304.8 29.21 0)
-			(effects
-				(font
-					(size 1.27 1.27)
-				)
-				(hide yes)
-			)
-		)
-		(property "Description" ""
-			(at 304.8 29.21 0)
-			(effects
-				(font
-					(size 1.27 1.27)
-				)
-				(hide yes)
-			)
-		)
-		(property "Manufacturer" "Generic"
-			(at 304.8 29.21 0)
-			(effects
-				(font
-					(size 1.27 1.27)
-				)
-				(hide yes)
-			)
-		)
-		(property "Part #" "Generic 0603 10k 1% Resistor"
-			(at 304.8 29.21 0)
-			(effects
-				(font
-					(size 1.27 1.27)
-				)
-				(hide yes)
-			)
-		)
-		(pin "1"
-		)
-		(pin "2"
-		)
-		(instances
-			(project "rocket2-afs"
-				(path "/bb02b74a-6e6c-4d52-9615-6a7971a5afcd"
-					(reference "R22")
-					(unit 1)
-				)
-			)
-		)
-	)
-	(symbol
 		(lib_id "power:GND")
 		(at 311.15 93.98 90)
@@
 					(unit 1)
 				)
-			)
-		)
-	)
-	(symbol
-		(lib_id "power:+3.3V")
-		(at 304.8 26.67 0)
-		(unit 1)
-		(exclude_from_sim no)
-		(in_bom yes)
-		(on_board yes)
-		(dnp no)
-		(property "Reference" "#PWR075"
-			(at 304.8 30.48 0)
-			(effects
-				(font
-					(size 1.27 1.27)
-				)
-				(hide yes)
-			)
-		)
-		(property "Value" "+3.3V"
-			(at 304.8 22.86 0)
-			(effects
-				(font
-					(size 1.27 1.27)
-				)
-			)
-		)
-		(property "Footprint" ""
-			(at 304.8 26.67 0)
-			(effects
-				(font
-					(size 1.27 1.27)
-				)
-				(hide yes)
-			)
-		)
-		(property "Datasheet" ""
-			(at 304.8 26.67 0)
-			(effects
-				(font
-					(size 1.27 1.27)
-				)
-				(hide yes)
-			)
-		)
-		(property "Description" ""
-			(at 304.8 26.67 0)
-			(effects
-				(font
-					(size 1.27 1.27)
-				)
-				(hide yes)
-			)
-		)
-		(pin "1"
-		)
-		(instances
-			(project "rocket2-afs"
-				(path "/bb02b74a-6e6c-4d52-9615-6a7971a5afcd"
-					(reference "#PWR075")
-					(unit 1)
-				)
