File: BUCK.kicad_sch (KiCad schematic)
At the start: 13 parts, among them U5 MP2338GTL-Z

Commit message: commit that was sent to jlcpcb
Parts:
- D11: value BLUE -> BLUE_LED
- L2: Part # (none) -> VLS6045EX-6R8M
- U5: Part # (none) -> MP2338GTL-P
Changed lines of the file:
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@@
 			)
 		)
-		(property "Description" ""
+		(property "Description" "Resistor, small US symbol"
 			(at 157.48 55.88 0)
 			(effects
@@
 			)
 		)
+		(property "Part #" "MP2338GTL-P"
+			(at 74.93 50.8 0)
+			(effects
+				(font
+					(size 1.27 1.27)
+				)
+				(hide yes)
+			)
+		)
 		(pin "8"
 		)
@@
 			)
 		)
-		(property "Datasheet" "https://www.digikey.com/en/products/detail/tdk-corporation/VLS6045EX-6R8M/5287380"
+		(property "Datasheet" "https://product.tdk.com/en/system/files/dam/doc/product/inductor/inductor/smd/catalog/inductor_commercial_power_vls6045ex_en.pdf"
 			(at 127 53.34 0)
 			(effects
@@
 		(property "Description" "Inductor, small symbol"
 			(at 127 53.34 0)
+			(effects
+				(font
+					(size 1.27 1.27)
+				)
+				(hide yes)
+			)
+		)
+		(property "Part #" "VLS6045EX-6R8M"
+			(at 127 53.34 90)
 			(effects
 				(font
@@
 			)
 		)
-		(property "Value" "BLUE"
+		(property "Value" "BLUE_LED"
 			(at 154.686 64.008 90)
 			(effects
