File: rc-plane.kicad_pcb (KiCad board)
At the start: 2 copper layers, 65 x 56 mm, 149 parts, among them J1 POWER, J2 ARMING_PLUG, J3 SMA, J4 E-MATCH_DROGUE, J5 SWD, J6 E-MATCH_RECOVERY, J8 E-MATCH_DROGUE, J9 HTSW-109-08-T-T-RA, Q1 Q_NMOS_GSD, Q2 Q_NMOS_GSD, Q3 BC547, Q4 Q_NMOS_GSD, Q5 Q_NMOS_GSD, Q6 Q_NMOS_GSD, Q7 Q_NMOS_GSD, U10 RASPBERRY_PI_4B_4GB, U12 MP2338GTL-Z, U13 MP2338GTL-Z, U5 MP2338GTL-Z, U8 BMM350, U9 USBLC6-2SC6, Y1 16MHz

Commit message: layout mostly done
Parts:
- removed C11: 120000uF, Capacitor_SMD:C_0603_1608Metric
- removed C13, C8: 12000uF, Capacitor_SMD:C_0603_1608Metric
- removed C16: C, Capacitor_SMD:C_0603_1608Metric
- removed MH1, MH2, MH3, MH4: M2.5, MountingHole:MountingHole_2.5mm
- removed R22: 10k, Resistor_SMD:R_0603_1608Metric
- added C1: 100nF, Capacitor_SMD:C_0603_1608Metric, B.Cu at (50.8, 134.1)
- C117, C14, C21, C25, C26, C27, C28, C29, C30, C31, C32, C33, C34, C36, C37, C38, C39, C4, C40, C41, C44, C45, C46, C47, C48, C49, C5, C50, C52, C53, C54, C55, C6, C7, D11, D12, D13, D4, D5, L2, L3, L4, Q1, Q2, Q4, Q5, Q6, Q7, R14, R15, R18, R19, R24, R25, R27, R30, R31, R32, R34, R35, R36, R37, R38, R39, R4, R40, R41, R42, R43, R46, R47, R48, R49, R5, R50, R51, R52, R53, R54, R55, R56, R57, R58, R59, R6, R60, R61, R7, R8, U11, U12, U13, U2, U46, U5, U6, U7, U8, U9, Y1: moved to B.Cu
- J8: value E-MATCH_DROGUE -> E-MATCH_BACKUP
- moved C32 281.3 mm to (324.0, 97.4)
- moved C30 273.1 mm to (319.8, 117.0)
- moved C29 272.7 mm to (316.5, 96.1), turned to 180 degrees
- moved C27 268.3 mm to (315.7, 116.0), turned to 180 degrees
- moved R27 262.4 mm to (318.7, 114.7), turned to 180 degrees
- moved R30 261.9 mm to (316.7, 114.7)
- moved C25 215.8 mm to (258.5, 140.9), turned to -90 degrees
- moved U6 206.7 mm to (320.3, 96.8), turned to 180 degrees
- moved C117 182.5 mm to (317.2, 118.0), turned to 180 degrees
- moved U7 176.8 mm to (255.3, 142.0), turned to 180 degrees
- moved C14 163.5 mm to (204.1, 105.8)
- moved R41 157.1 mm to (324.0, 95.8)
- moved R53 156.0 mm to (89.8, 71.5), turned to 180 degrees
- moved U12 151.6 mm to (93.6, 72.2), turned to 180 degrees
- moved R42 149.8 mm to (316.5, 97.8), turned to 180 degrees
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Connections:
- D1 pad 1: (no net) -> BATTERY
- D1 pad 2: (no net) -> GND
- J2 pad 1: POWER -> BATTERY
- J9 pad 01: ELEV_PWM1 -> GND
- J9 pad 03: GND -> ELEV_PWM1
- J9 pad 04: RUDD_PWM2 -> GND
- J9 pad 06: GND -> RUDD_PWM2
- J9 pad 07: AIL_L_PWM3 -> GND
- J9 pad 09: GND -> AIL_L_PWM3
- J9 pad 10: AIL_R_PWM4 -> GND
- J9 pad 12: GND -> AIL_R_PWM4
- J9 pad 13: FLAP_L_PWM5 -> GND
- J9 pad 15: GND -> FLAP_L_PWM5
- J9 pad 16: FLAP_R_PWM6 -> GND
- J9 pad 18: GND -> FLAP_R_PWM6
- J9 pad 19: ESC_PWM0 -> GND
- J9 pad 21: GND -> ESC_PWM0
- U46 pad 9: (no net) -> GND
Routing:
- net GND: track 0.00 -> 130.7 mm, vias 0 -> 82
- net BATTERY: track 0.00 -> 97.1 mm
- net FLAP_R_PWM6: track 0.00 -> 69.3 mm
- net ESC_PWM0: track 0.00 -> 68.1 mm
- net FLAP_L_PWM5: track 0.00 -> 66.3 mm
- net +3.3V: track 0.00 -> 62.9 mm, vias 0 -> 24
- net AIL_L_PWM3: track 0.00 -> 50.8 mm
- net ARM_POWER: track 0.00 -> 48.1 mm
- net AIL_R_PWM4: track 0.00 -> 46.9 mm, vias 0 -> 1
- net RUDD_PWM2: track 0.00 -> 42.4 mm, vias 0 -> 1
- net ELEV_PWM1: track 0.00 -> 39.0 mm
- net VBUS: track 0.00 -> 37.2 mm, vias 0 -> 4
- net USB_D-: track 0.00 -> 35.6 mm
- net USB_D+: track 0.00 -> 34.9 mm
- net DEBUG_SWCLK: track 0.00 -> 33.2 mm, vias 0 -> 1
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Other:
- copper layers 2 -> 4

Commit message: PCB done
Parts:
- removed D6: 1N4148WT, Diode_SMD:D_SOD-523
- removed Q3: BC547, Package_TO_SOT_THT:TO-92_Inline
- removed R11: 180, Resistor_SMD:R_0603_1608Metric
- added G***: LOGO, LOGO, F.Cu at (107.3, 61.5)
- C15, C42: moved to B.Cu
- R1: value 27k -> 33k; moved to B.Cu
- R3: value 6k -> 10k; moved to B.Cu
- moved C30 219.2 mm to (107.2, 63.4), turned to -90 degrees
- moved C117 218.6 mm to (106.2, 60.8), turned to 90 degrees
- moved U8 217.0 mm to (107.8, 61.3), turned to 90 degrees
- moved R27 215.7 mm to (109.5, 62.3), turned to 90 degrees
- moved C27 215.1 mm to (108.2, 59.3), turned to 90 degrees
- moved R30 214.2 mm to (109.5, 60.3), turned to -90 degrees
- moved C32 196.3 mm to (130.4, 64.8), turned to 180 degrees
- moved R41 192.9 mm to (133.6, 64.8)
- moved U6 192.5 mm to (130.9, 62.2), turned to 90 degrees
- moved R42 190.7 mm to (129.9, 58.4), turned to 90 degrees
- moved C29 188.7 mm to (131.6, 58.4), turned to 90 degrees
- moved R40 150.3 mm to (117.9, 75.3), turned to -90 degrees
- moved C25 149.0 mm to (123.0, 79.0), turned to 180 degrees
- moved U7 148.9 mm to (121.9, 75.8), turned to 90 degrees
- moved R3 137.2 mm to (135.6, 58.4)
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Connections:
- U11 pad 29: EN_5V -> EN_SERVO
Routing:
- net NRST: track 0.00 -> 110.7 mm, vias 0 -> 3
- net VBUS_SENS: track 1.90 -> 63.4 mm, vias 0 -> 2
- net ESC_PWM0: track 68.1 -> 119.1 mm, vias 0 -> 3
- net FLAP_R_PWM6: track 69.3 -> 118.4 mm, vias 0 -> 3
- net LED_STANDBY: track 6.26 -> 54.1 mm, vias 1 -> 4
- net DROGUE: track 2.38 -> 49.2 mm, vias 0 -> 2
- net MEM_MISO: track 0.00 -> 44.0 mm, vias 0 -> 3
- net LED_FLIGHT: track 6.19 -> 49.1 mm, vias 1 -> 4
- net LED_STORAGE: track 6.29 -> 49.0 mm, vias 1 -> 4
- net LED_ARMED: track 6.24 -> 46.8 mm, vias 1 -> 4
- net RADIO_CS: track 20.1 -> 59.5 mm, vias 1 -> 3
- net FLAP_L_PWM5: track 66.3 -> 104.4 mm, vias 0 -> 2
- net DROGUE_CONT: track 2.31 -> 40.1 mm, vias 0 -> 2
- net EN_SERVO: track 8.55 -> 45.5 mm, vias 2 -> 5
- net RECOVERY: track 2.38 -> 37.3 mm, vias 0 -> 2
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- added copper zone on B.Cu, net +3.3V
- added copper zone on In2.Cu, net +3.3V
- added copper zone on B.Cu, net +5V
- added copper zone on B.Cu, net +5V_SERVO
- added copper zone on B.Cu, net BATTERY
- added copper zone on F.Cu, net BATTERY
- added copper zone on B.Cu, net GND
- added copper zone on F.Cu, net GND
- added copper zone on In1.Cu, net GND
- added copper zone on B.Cu, net VCC
Other:
- board text added: "+"
- board text added: "ARM"
- board text added: "BACKUP"
- board text added: "BATTERY"
- board text added: "DROGUE"
- board text added: "ELEVATOR RUDDER AILERON LEFT AILERON RIGHT FLAP LEFT FLAP RIGHT ELEC SPEED CONTR LED LEFT LED RIGHT"
- board text added: "MAIN"
- board text added: "Pi Flight Sensor Hat By: Robert Woo YoungWoo Chang Quynh Nguyen"
- board text added: "STANDBY STORAGE FLIGHT ARMED"
- board text added: "SWD"
- board text added: "USB C"

Commit message: Added gerber, BOM, and parts list csv files for fab.
Connections:
- U10 pad S1: GND -> SHIELD_1
- U10 pad S2: GND -> SHIELD_3
- U10 pad S3: GND -> SHIELD
- U10 pad S4: GND -> SHIELD_2
Changed lines of the file:
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@@
 		(allow_soldermask_bridges_in_footprints no)
 		(tenting front back)
+		(aux_axis_origin 78 105)
 		(pcbplotparams
 			(layerselection 0x00000000_00000000_55555555_5755f5ff)
@@
 			(outputformat 1)
 			(mirror no)
-			(drillshape 1)
+			(drillshape 0)
 			(scaleselection 1)
-			(outputdirectory "")
+			(outputdirectory "Fab/")
 		)
 	)
@@
 	(net 146 "unconnected-(U2-DIO3-Pad11)")
 	(net 147 "RADIO_DIO1")
+	(net 148 "SHIELD")
+	(net 149 "SHIELD_1")
+	(net 150 "SHIELD_2")
+	(net 151 "SHIELD_3")
 	(footprint "Resistor_SMD:R_0603_1608Metric"
 		(layer "F.Cu")
@@
 			(layers "*.Cu" "*.Mask")
 			(remove_unused_layers no)
-			(net 2 "GND")
+			(net 149 "SHIELD_1")
 			(pinfunction "SHIELD")
-			(pintype "power_in")
+			(pintype "power_in+no_connect")
 			(solder_mask_margin 0.102)
 		)
@@
 			(layers "*.Cu" "*.Mask")
 			(remove_unused_layers no)
-			(net 2 "GND")
+			(net 151 "SHIELD_3")
 			(pinfunction "SHIELD")
-			(pintype "power_in")
+			(pintype "power_in+no_connect")
 			(solder_mask_margin 0.102)
 		)
@@
 			(layers "*.Cu" "*.Mask")
 			(remove_unused_layers no)
-			(net 2 "GND")
+			(net 148 "SHIELD")
 			(pinfunction "SHIELD")
-			(pintype "power_in")
+			(pintype "power_in+no_connect")
 			(solder_mask_margin 0.102)
 		)
@@
 			(layers "*.Cu" "*.Mask")
 			(remove_unused_layers no)
-			(net 2 "GND")
+			(net 150 "SHIELD_2")
 			(pinfunction "SHIELD")
-			(pintype "power_in")
+			(pintype "power_in+no_connect")
 			(solder_mask_margin 0.102)
 		)
@@
 			(unlocked yes)
 			(layer "B.SilkS")
-			(hide yes)
 			(effects
 				(font
@@
 			(unlocked yes)
 			(layer "B.SilkS")
-			(hide yes)
 			(effects
 				(font
@@
 			(unlocked yes)
 			(layer "B.SilkS")
-			(hide yes)
 			(effects
 				(font

Commit message: commit that was sent to jlcpcb
Parts:
- removed R34, R37, R8: 1, Resistor_SMD:R_0603_1608Metric
- added G***: LOGO, LOGO, F.Cu at (106.9, 89.6)
- added R11: 10, Resistor_SMD:R_0603_1608Metric, B.Cu at (141.6, 61.6)
- D10, D11, D12, D13: value BLUE -> BLUE_LED
- D5: value D_LIPO -> SS34
- J7: value ~ -> USB4105-GF-A
- R58: value 191k -> 200k
- R59: value 49.9k -> 80k
- U11: value ~ -> STM32F105RCT6
- U2: value ~ -> RFM95W
- U3: value ~ -> SAM-M8Q-0
- U46: value ~ -> W25N01GVZEIG TR
- U6: value ~ -> BMI088
- U7: value ~ -> MS5607-02BA03
- moved C43 6.84 mm to (97.6, 69.0), turned to 180 degrees
- turned R50 to 180 degrees
Connections:
- J2 pad 2: ARM_POWER -> Net-(J2-Pin_2)
- Q2 pad 2: Net-(Q2-S) -> GND
- Q4 pad 2: Net-(Q4-S) -> GND
- Q7 pad 2: Net-(Q7-S) -> GND
- R1 pad 1: ARM_POWER -> Net-(J2-Pin_2)
- U11 pad 37: BUZZER -> RADIO_DIO1
- U11 pad 6: unconnected-(U11-PD1-Pad6) -> RADIO_DIO0
Routing:
- net RADIO_DIO0: track 0.00 -> 43.7 mm, vias 0 -> 2
- net RADIO_DIO1: track 0.00 -> 35.1 mm, vias 0 -> 2
- net GND: track 145.4 -> 156.0 mm, vias 104 -> 105
- net Net-(J2-Pin_2): track 0.00 -> 6.99 mm
- net Net-(U12-SS): track 0.56 -> 7.12 mm
- net ARM_POWER: track 47.7 -> 41.7 mm
- net EN_SERVO: track 45.5 -> 49.9 mm
- net Net-(Q4-S): track 1.79 -> 0.00 mm
- net Net-(Q7-S): track 1.77 -> 0.00 mm
- net Net-(Q2-S): track 1.76 -> 0.00 mm
- net Net-(U12-PG): track 7.80 -> 9.43 mm
- net +3.3V: vias 77 -> 67
