File: rc-plane.kicad_sch (KiCad schematic)
At the start: 104 parts, among them J1 POWER, J2 ARMING_PLUG, J3 SMA, J4 E-MATCH_DROGUE, J5 SWD, J6 E-MATCH_RECOVERY, J8 E-MATCH_BACKUP, J9 HTSW-109-08-T-T-RA, Q1 Q_NMOS_GSD, Q2 Q_NMOS_GSD, Q3 BC547, Q4 Q_NMOS_GSD, Q5 Q_NMOS_GSD, Q6 Q_NMOS_GSD, Q7 Q_NMOS_GSD, U10 RASPBERRY_PI_4B_4GB, U8 BMM350, U9 USBLC6-2SC6, Y1 16MHz

Commit message: PCB done
Parts:
- removed D6: 1N4148WT, Diode_SMD:D_SOD-523, symbol Diode:1N4148WT
- removed LS1: CMT-7525S-SMT, CMT-7525S-SMT:CUI_CMT-7525S-SMT, symbol CMT-7525S-SMT:CMT-7525S-SMT
- removed Q3: BC547, Package_TO_SOT_THT:TO-92_Inline, symbol Transistor_BJT:BC547
- removed R11: 180, Resistor_SMD:R_0603_1608Metric, symbol Device:R_Small_US
- removed R22: 10k, Resistor_SMD:R_0603_1608Metric, symbol Device:R_Small_US
- R1: value 27k -> 33k
- R3: value 6k -> 10k
Connections:
- net EN_5V is gone; now on net EN_SERVO: U11.29 (PB10)
Other:
- note added: "LEDS"
- note removed: "LEDS + PIEZO BUZZER"
- note removed: "Reset Pin cannot be driven HIGH"

Commit message: Added gerber, BOM, and parts list csv files for fab.
Connections:
- net GND: no longer U10.S1 (SHIELD), U10.S2 (SHIELD), U10.S3 (SHIELD), U10.S4 (SHIELD)
- new net SHIELD: U10.S1 (SHIELD), U10.S2 (SHIELD), U10.S3 (SHIELD), U10.S4 (SHIELD)
- no-connect marks 44 -> 45
Changed lines of the file:
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@@
-	)
-	(junction
-		(at 187.96 97.79)
-		(diameter 0)
-		(color 0 0 0 0)
 	)
 	(junction
@@
 	)
 	(no_connect
+		(at 187.96 95.25)
+	)
+	(no_connect
 		(at 147.32 64.77)
 	)
@@
 		)
 		(stroke
-			(width 0)
-			(type default)
-		)
-	)
-	(wire
-		(pts
-			(xy 187.96 95.25) (xy 187.96 97.79)
-		)
-		(stroke

Commit message: commit that was sent to jlcpcb
Parts:
- removed R34, R37, R8: 1, Resistor_SMD:R_0603_1608Metric, symbol Device:R_Small_US
- added R11: 10, Resistor_SMD:R_0603_1608Metric, symbol Device:R_Small_US
- D1: Part # (none) -> SMBJ26CA
- D10: value BLUE -> BLUE_LED
- D4: Part # (none) -> SS34
- D5: value D_LIPO -> SS34; Part # (none) -> SS34
- J2, J4, J6, J8, U10: now left out of the parts list
- J3: now not fitted; now left out of the parts list
- J5: Part # Generic 2x05 P1.27mm Vertical Pin Header SMD -> 4048
- J7: value ~ -> USB4105-GF-A
- J9: Part # (none) -> HTSW-109-08-T-T-RA
- Q1, Q2, Q4, Q5, Q6, Q7: Part # PMV30UN2 -> WST3408
- R58: value 191k -> 200k
- R59: value 49.9k -> 80k
- U11: value ~ -> STM32F105RCT6
- U2: value ~ -> RFM95W; now not fitted; now left out of the parts list
- U3: value ~ -> SAM-M8Q-0; Part # SAM-M8Q -> SAM-M8Q-0
- U46: value ~ -> W25N01GVZEIG TR
- U6: value ~ -> BMI088
- U7: value ~ -> MS5607-02BA03; Part # MS560702BA03-50 -> MS5607-02BA03
- U8: Part # (none) -> BMM350
- Y1: Part # ECS-1633-160-BN-TR -> ECS-1633-120-BN-TR
Connections:
- net BUZZER is gone; now on net RADIO_DIO1: U11.37 (PC6)
- net ARM_POWER: now also R11.1; no longer J2.2 (Pin_2), R1.1
- net GND: now also Q2.2 (S), Q4.2 (S), Q7.2 (S)
- net RADIO_DIO0: now also U11.6 (PD1)
- new net: J2.2 (Pin_2), R1.1, R11.2
- no-connect marks 45 -> 44
Other:
- moved on the sheet: C14, C25, C55, D1, J1, J2, J4, J5, J6, J8, J9, Q1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
