File: KICAD PCB/rc-plane.kicad_sch (KiCad schematic)
At the start: 97 parts, among them J1 POWER, J2 ARMING_PLUG, J3 SMA, J4 E-MATCH_DROGUE, J5 SWD, J6 E-MATCH_RECOVERY, J7 USB4105-GF-A, J8 E-MATCH_BACKUP, J9 HTSW-109-08-T-T-RA, Q1 Q_NMOS_GSD, Q2 Q_NMOS_GSD, Q4 Q_NMOS_GSD, Q5 Q_NMOS_GSD, Q6 Q_NMOS_GSD, Q7 Q_NMOS_GSD, U10 RASPBERRY_PI_4B_4GB, U11 STM32F105RCT6, U2 RFM95W, U3 SAM-M8Q-0, U46 W25N01GVZEIG TR, U6 BMI088, U7 MS5607-02BA03, U8 BMM350, U9 USBLC6-2SC6, Y1 16MHz

Commit message: working on rev2 on the board, deving out code for flight for stm32 software
Parts:
- removed J2: ARMING_PLUG, TerminalBlock:TerminalBlock_bornier-2_P5.08mm, symbol Connector:Conn_01x02_Socket
- removed J4: E-MATCH_DROGUE, TerminalBlock:TerminalBlock_bornier-2_P5.08mm, symbol Connector:Conn_01x02_Socket
- removed J6: E-MATCH_RECOVERY, TerminalBlock:TerminalBlock_bornier-2_P5.08mm, symbol Connector:Conn_01x02_Socket
- removed J8: E-MATCH_BACKUP, TerminalBlock:TerminalBlock_bornier-2_P5.08mm, symbol Connector:Conn_01x02_Socket
- removed Q7: Q_NMOS_GSD, Package_TO_SOT_SMD:TSOT-23, symbol Device:Q_NMOS_GSD
- removed R31: 100k, Resistor_SMD:R_0603_1608Metric, symbol Device:R_Small_US
- added C13: 0.33uF, Capacitor_SMD:C_0603_1608Metric, symbol Device:C_Small
- added C16, C18: 0.1uF, Capacitor_SMD:C_0603_1608Metric, symbol Device:C_Small
- added J10: Conn_01x06_Socket, TerminalBlock:TerminalBlock_Xinya_XY308-2.54-6P_1x06_P2.54mm_Horizontal, symbol Connector:Conn_01x06_Socket
- added J2: 2.54mm 3x08 header, UCIRP-KiCAD-Lib:HX PZ2.54-3x8P ZZ 3x08 2.54mm THT header, symbol UCIRP-KiCAD-Lib:HX PZ2.54-3x8P ZZ
- added J4: ALARM, UCIRP-KiCAD-Lib:XDCR_SMT-0540-S-R, symbol Connector:Conn_01x02_Pin
- added R12, R22: 80k, Resistor_SMD:R_0603_1608Metric, symbol Device:R_Small_US
- added R13, R8: 200k, Resistor_SMD:R_0603_1608Metric, symbol Device:R_Small_US
- added R37: 100, Resistor_SMD:R_0402_1005Metric, symbol Device:R_Small_US
- added U1: MAX11614, Package_SO:QSOP-16_3.9x4.9mm_P0.635mm, symbol Analog_ADC:MAX11614
- added U33: AS78L05RTR, Package_TO_SOT_SMD:SOT-89-3, symbol UCIRP-KiCAD-Lib:Generic_Regulator_InputGroundOutput
- J1: Part # Generic Horizontal TH P5.08mm Screw Fastened -> XT60PW-F
- J3, U2: now fitted
- R35: value 1k -> 2k; Manufacturer Generic -> (none); Part # Generic 0603 1k 1% Resistor -> (none)
- R36: value 10k -> 10K; footprint Resistor_SMD:R_0603_1608Metric -> Resistor_SMD:R_0402_1005Metric; Part # Generic 0603 10k 1% Resistor -> Generic RES SMD 10K OHM 1% 1/4W 0402
- R38: value 100 -> 22R; footprint Resistor_SMD:R_0603_1608Metric -> Resistor_SMD:R_0402_1005Metric; Part # Generic 0603 100 1% Resistor -> Generic RES SMD 4.7K OHM 1% 1/4W 0402
- R39: value 10k -> 22R; footprint Resistor_SMD:R_0603_1608Metric -> Resistor_SMD:R_0402_1005Metric; Part # Generic 0603 10k 1% Resistor -> Generic RES SMD 4.7K OHM 1% 1/4W 0402
- R54: value 100k -> 22R; footprint Resistor_SMD:R_0603_1608Metric -> Resistor_SMD:R_0402_1005Metric; Manufacturer (none) -> Generic; Part # (none) -> Generic RES SMD 4.7K OHM 1% 1/4W 0402
Connections:
- net Buck1/FB is gone; now on net +5V: C21.2, R32.1, R43.1
- net +3.3V: now also J4.1 (Pin_1); no longer R35.1
- net ARM_CONT: now also U1.11 (AIN6); no longer U11.11 (PC3)
- net ARM_POWER: now also J10.3 (Pin_3), J10.5 (Pin_5)
- net BATTERY: now also J1.2 (Pin_2), C13.2, J10.1 (Pin_1), J2.10 (Pin_10), J2.11 (Pin_11), J2.12 (Pin_12), J2.13 (Pin_13), J2.14 (Pin_14), J2.9 (Pin_9), R13.1, R8.1, U33.1 (VIN); no longer J1.1 (Pin_1)
- net GND: now also J1.1 (Pin_1), R36.1, C13.1, C16.2, C18.1, J2.1 (Pin_1), J2.2 (Pin_2), J2.3 (Pin_3), J2.4 (Pin_4), J2.5 (Pin_5), J2.6 (Pin_6), J2.7 (Pin_7), J2.8 (Pin_8), R12.2, R22.2, U1.15 (GND), U33.2 (GND); no longer J1.2 (Pin_2), R36.2, R39.2, R54.2
- net IMU_MISO: now also U11.22 (PA6); no longer U11.23 (PA7)
- net IMU_MOSI: now also U11.23 (PA7); no longer U11.22 (PA6)
- net MAG_INT: no longer U11.40 (PC9)
- net MAG_SCL: now also U1.13 (SCL)
- net MAG_SDA: now also U1.14 (SDA)
- net MEM_HOLD: no longer U11.50 (PA15)
- net MEM_MISO: now also R39.2; no longer U11.56 (PB4)
- net MEM_MOSI: now also R54.2; no longer U11.57 (PB5)
- net MEM_SCK: now also R38.2; no longer U11.55 (PB3)
- net MEM_WP: no longer U11.43 (PA10)
- net RADIO_DIO0: no longer U11.6 (PD1)
- net RADIO_DIO1: no longer U11.37 (PC6)
- net MAIN-: now reaches Q4.3 (D), Q5.1 (G), R18.1
- net MAIN-: now also J10.6 (Pin_6)
- net at Q6.1 (G): now also R37.2; no longer R36.1
- net ARM-: now reaches R1.1, R11.2
- net ARM-: now also J10.2 (Pin_2)
- net DROGUE-: now reaches Q1.1 (G), Q2.3 (D), R5.1
- net DROGUE-: now also J10.4 (Pin_4)
- net at R38.1: now also U11.55 (PB3)
- removed net BACKUP: R38.2, R39.1, U11.3 (PC14)
- removed net BACKUP_CONT: Q6.3 (D), R35.2, U11.2 (PC13)
- net EN_PI: no longer names the net of U11.30 (PB11)
- net EN_SERVO: no longer names the net of U11.29 (PB10)
- net EN_SERVO: no longer R54.1
- net RECOVERY renamed MAIN
- net MAIN: no longer U11.10 (PC2)
- net RECOVERY_CONT renamed MAIN_CONT
- net MAIN_CONT: no longer U11.9 (PC1)
- new net: J4.2 (Pin_2), Q6.3 (D)
- new net: C18.2, R35.1
- new net: R35.2, U1.1 (REF)
- new net: R39.1, U11.56 (PB4)
- new net: R54.1, U11.57 (PB5)
- new net +5V_ADC: C16.1, J2.15 (Pin_15), J2.16 (Pin_16), U1.16 (Vdd), U33.3 (VOUT)
- new net ADC_AIN1: J2.17 (Pin_17)
- new net ADC_AIN2: J2.18 (Pin_18)
- new net ADC_AIN3: J2.19 (Pin_19)
- new net ADC_AIN4: J2.20 (Pin_20)
- new net ADC_AIN5: J2.21 (Pin_21)
- new net ADC_AIN6: J2.22 (Pin_22)
- new net AI_DIFF +: J2.23 (Pin_23)
- new net AI_DIFF -: J2.24 (Pin_24)
- new net ALARM: R36.2, R37.1
- new net Buck/EN: R13.2, R22.1
- new net Buck1/EN: R12.1, R8.2
- new net Differential-ADC/AO: U1.12 (AIN7)
- new net Single_Ended_ADC/OUT: U1.5 (AIN0)
- new net Single_Ended_ADC1/OUT: U1.6 (AIN1)
- new net Single_Ended_ADC2/OUT: U1.7 (AIN2)
- new net Single_Ended_ADC3/OUT: U1.8 (AIN3)
- new net Single_Ended_ADC4/OUT: U1.9 (AIN4)
- new net Single_Ended_ADC5/OUT: U1.10 (AIN5)
- no-connect marks 44 -> 45
Other:
- added sheet Differential-ADC (loadcell.kicad_sch)
- added sheet Single_Ended_ADC (pt.kicad_sch)
- added sheet Single_Ended_ADC1 (pt.kicad_sch)
- added sheet Single_Ended_ADC2 (pt.kicad_sch)
- added sheet Single_Ended_ADC3 (pt.kicad_sch)
- added sheet Single_Ended_ADC4 (pt.kicad_sch)
- added sheet Single_Ended_ADC5 (pt.kicad_sch)
- note added: "ARMING PLUG, DROGUE AND MAIN PARACHUTE IGNITION"
- note added: "EXTERNAL ADC"
- note added: "EXTERNAL ADC HEADER"
- note added: "LEDS + ALARM"
- note removed: "ARMING PLUG"
- note removed: "DROGUE, MAIN, AND BACKUP PARACHUTE IGNITION"
- note removed: "LEDS"
- note removed: "always enabled"
- moved on the sheet: C1, C14, C21, C25, C33, C34, C4, C42, C48, C5, C55, C6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

Commit message: moved to stm32cube vscode extension, v2.0 purchased
Parts:
- J4: Manufacturer Same Sky -> (none); Part # CMI-0955-03TH -> SMT-0540-S-R
- J5: Part # 4048 -> X1321WVS-2x05J-C40D53
- R12, R22, R59: value 80k -> 82k
Connections:
- net +5V: no longer C21.2, R32.1, R43.1
- net GPS_INT: now also U11.2 (PC13)
- net GPS_RESET: now also U11.40 (PC9)
- net GPS_SAFEBOOT: now also U11.3 (PC14)
- net MAG_INT: now also U11.11 (PC3)
- net MAIN: now also U11.10 (PC2)
- net MAIN_CONT: now also U11.9 (PC1)
- net RADIO_DIO0: now also U11.29 (PB10)
- net RADIO_DIO1: now also U11.30 (PB11)
- net RADIO_nRST: now also U11.37 (PC6)
- net MAG_SCL renamed SCL
- net MAG_SDA renamed SDA
- new net Buck1/FB: C21.2, R32.1, R43.1
- no-connect marks 45 -> 47
Other:
- note added: "5V for ADC"
- note added: "Rev changes from v1 to v2: Miso and Mosi and backwards on IMU PD1 has to be floating Added external, I2C ADC"
- note removed: "ACD1_IN13"
- note removed: "Rev changes: Miso and Mosi and backwards on IMU PD1 has to be floating"
- moved on the sheet: C13, C16, C18, R35, U33, U9
